Commit message: added cams, got new kickers working with old box photoeye demo

File: urdf/kicker/side_kicker.urdf (robot description, URDF)
Before this commit: robot onshape, 2 links, 1 joints
Links:
- removed link base_link
- removed link kicker_link
- added link kicker_arm, mass 0; collision mesh filename=package://urdf/kicker/kicker_arm.stl; visual mesh filename=package://urdf/kicker/kicker_arm.stl
- added link kicker_base, mass 0; collision mesh filename=package://urdf/kicker/kicker_base.stl; visual mesh filename=package://urdf/kicker/kicker_base.stl
Joints:
- joint kicker_joint: child kicker_link -> kicker_arm; limit lower=0 upper=1.0471975511965976313 effort=1 velocity=20 -> lower=0 upper=1.1999999999999999556 effort=1 velocity=20; origin xyz=4.336808689942017736e-19 3.9239621782441154511e-19 0.025000000000000001388 rpy=3.141592653589793116 -0 0 -> xyz=0.012499999999999955591 -0.39999999999999991118 0.15000000000000007772 rpy=1.570796326794896558 -0 1.570796326794896558; parent base_link -> kicker_base; type revolute -> prismatic

Commit message: merged ros package and isaac extension, tested package basics

File: urdf/kicker/side_kicker.urdf (robot description, URDF)
Before this commit: robot onshape, 2 links, 1 joints
Links:
- link kicker_arm: geometry collision mesh filename=package://isaac_cam_conveyor/urdf/kicker/kicker_arm.stl; visual mesh filename=package://isaac_cam_conveyor/urdf/kicker/kicker_arm.stl
- link kicker_base: geometry collision mesh filename=package://isaac_cam_conveyor/urdf/kicker/kicker_base.stl; visual mesh filename=package://isaac_cam_conveyor/urdf/kicker/kicker_base.stl
